Commit message: Add trackball to urdf

File: offboard/src/rviz_vis/urdf/tactile-odom-drone.urdf (robot description, URDF)
Before this commit: robot am, 4 links, 3 joints
Links:
- link ee: geometry collision sphere radius=0.01
- link link2: geometry collision box size=0.07 0.05 0.01; visual mesh filename=package://rviz_vis/meshes/Link2Assembly.dae scale=0.001 0.001 0.001
Joints:
- joint ee_connector: origin xyz=0.0 0.0 0.02 rpy=0 0 0 -> xyz=0.0 0.0 0.028 rpy=0 0 0
